File: hack.sch (EAGLE design)
At the start: 40 parts, among them IC1 NUF2221W1T2G, IC3 LDO, IC4 ATSAMR21G, J1 USB-micro, SW1 SPST3.5X6MM, X1 TSX-3225 16 MHz, X2 MC-306 32.768 KHz

Commit message: Second commit
Parts:
- added B1: BALUN, hack:BALUN
- added C18, C19: 22pF, jack:C-EU
- added JP4: (no value), pinhead:PINHD-1X2
Connections:
- net N$4 renamed AVDD
- removed net 1: JP1.5
- removed net 14: JP2.15
- removed net 15: JP2.14
- removed net 16: JP2.13
- removed net 2: JP1.4
- removed net 3: JP1.3
- removed net 37: JP1.12
- removed net 38: JP1.11
- removed net 39: JP1.10
- removed net 41: JP1.8
- removed net 47: JP1.2
- removed net 48: JP1.1
- new net N$5: B1.B1, C18.2
- new net N$6: B1.B2, C19.2
- new net PA04: IC4ATSAMR21G.PA04/A, JP1.3
- new net PA05: IC4ATSAMR21G.PA05/A, JP1.2
- new net PA06: IC4ATSAMR21G.PA06/A, JP1.1
- new net PA07: IC4ATSAMR21G.PA07/A, JP2.15
- new net PA08: IC4ATSAMR21G.PA08/D, JP2.14
- new net PA09: IC4ATSAMR21G.PA09/D, JP2.13
- new net PA27: IC4ATSAMR21G.PA27/D, JP1.10
- new net PA28: IC4ATSAMR21G.PA28/D, JP1.8
- new net PB02: IC4ATSAMR21G.PB02/A, JP1.5
- new net PB03: IC4ATSAMR21G.PB03/A, JP1.4
- new net PB22: IC4ATSAMR21G.PB22/D, JP1.12
- new net PB23: IC4ATSAMR21G.PB23/D, JP1.11
- new net RFN: C18.1, IC4ATSAMR21G.RFN
- new net RFP: C19.1, IC4ATSAMR21G.RFP
- new net SMA: B1.UN, JP4.1
- net !RESET: now also IC4ATSAMR21G.!RESET
- net GND: now also B1.GND, B1.GND/DC, B1.P$1, JP4.2
Other:
- moved on the sheet: IC4ATSAMR21G

Commit message: Finishing layout, added PCB antenna
Parts:
- removed JP2: (no value), pinhead:PINHD-1X17
- removed JP3: (no value), pinhead:PINHD-1X8
- removed JP4: (no value), pinhead:PINHD-1X2
- added ANT1: PCB-ANTENNA, hack:PCB-ANTENNA
- added JP5: (no value), pinhead:PINHD-1X5
- added JP6: (no value), pinhead:PINHD-1X10
Connections:
- removed net 10: JP3.5
- removed net 11: JP3.6
- removed net 12: JP3.7
- removed net 13: JP3.8
- removed net 19: JP2.12
- removed net 20: JP2.11
- removed net 21: JP2.10
- removed net 22: JP2.9
- removed net 25: JP2.8
- removed net 26: JP2.7
- removed net 27: JP2.6
- removed net 28: JP2.5
- removed net 29: JP2.4
- removed net 30: JP2.3
- removed net 31: JP2.2
- removed net 32: JP2.1, R5.2
- removed net 4: JP3.1
- removed net 7: JP3.3
- removed net 8: JP3.4
- removed net 9: JP3.2
- removed net GNDANA: JP2.17, R4.2
- removed net SMA: B1.UN, JP4.1
- new net N$4: ANT1.ANT, B1.UN
- new net PA12: IC4ATSAMR21G.PA12/D, JP6.1
- new net PA13: IC4ATSAMR21G.PA13/D, JP6.2
- new net PA14: IC4ATSAMR21G.PA14/D/XIN, JP6.3
- new net PA15: IC4ATSAMR21G.PA15/D/XOUT, JP6.4
- new net PA16: IC4ATSAMR21G.PA16/D, JP6.5
- new net PA17: IC4ATSAMR21G.PA17/D, JP6.6
- new net PA18: IC4ATSAMR21G.PA18/D, JP6.7
- new net PA19: IC4ATSAMR21G.PA19/D, JP6.8
- new net PA22: IC4ATSAMR21G.PA22/D, JP6.9
- new net PA23: IC4ATSAMR21G.PA23/D, JP6.10, R5.2
- net AGND: now also JP5.1, R4.2
- net GND: now also ANT1.GND; no longer JP4.2
- net PA07: now also JP5.3; no longer JP2.15
- net PA08: now also JP5.4; no longer JP2.14
- net PA09: now also JP5.5; no longer JP2.13
- net VDDANA: now also JP5.2; no longer JP2.16

Commit message: Third commit
Changed cutout of PCB so that one side hosts the antenna; moved part of
the header to the right side (use a female receptacle instead of a male
header to retain breadboard usability)
Changed lines of the file:
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@@
-</segment>
-</net>
-<net name="NC" class="0">
-<segment>
-<wire x1="107.95" y1="-7.62" x2="113.03" y2="-7.62" width="0.1524" layer="91"/>
-<label x="113.03" y="-7.62" size="1.27" layer="95" xref="yes"/>
-</segment>
-<segment>
-<wire x1="107.95" y1="-5.08" x2="113.03" y2="-5.08" width="0.1524" layer="91"/>
-<label x="113.03" y="-5.08" size="1.27" layer="95" xref="yes"/>
 </segment>
 </net>

Commit message: Added impedance controlled microstrips
Added impedance controlled microstrips (diff. impedance of 100 Ohms from
chip to balun, single ended impedance of 50 Ohms from balun to antenna)
Parts:
- removed C18: 22pF, jack:C-EU
Connections:
- removed net N$4: ANT1.ANT, B1.UN
- removed net N$6: B1.B2, C19.2
- new net ANT: ANT1.ANT, C19.2
- net N$5: now also B1.UN, C19.1; no longer B1.B1, C18.2
- net RFN: now also B1.B1; no longer C18.1
- net RFP: now also B1.B2; no longer C19.1
Other:
- moved on the sheet: C19
Changed lines of the file:
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@@
 <part name="GND12" library="cortexm0" deviceset="GND" device=""/>
 <part name="B1" library="hack" deviceset="BALUN" device=""/>
-<part name="C18" library="jack" deviceset="C-EU" device="" value="22pF"/>
 <part name="C19" library="jack" deviceset="C-EU" device="" value="22pF"/>
 <part name="GND13" library="cortexm0" deviceset="GND" device=""/>
@@
 <instance part="GND12" gate="G$1" x="81.28" y="-78.74"/>
 <instance part="B1" gate="G$1" x="73.66" y="-15.24"/>
-<instance part="C18" gate="G$1" x="86.36" y="-5.08" rot="MR90"/>
-<instance part="C19" gate="G$1" x="86.36" y="-25.4" rot="MR90"/>
+<instance part="C19" gate="G$1" x="63.5" y="-5.08" rot="MR90"/>
 <instance part="GND13" gate="G$1" x="81.28" y="-15.24" rot="R90"/>
 <instance part="GND14" gate="G$1" x="73.66" y="-30.48"/>
-<instance part="GND15" gate="G$1" x="55.88" y="-5.08"/>
+<instance part="GND15" gate="G$1" x="50.8" y="-3.81"/>
 <instance part="JP5" gate="A" x="105.41" y="2.54" rot="MR0"/>
 <instance part="JP6" gate="A" x="105.41" y="-20.32" rot="MR0"/>
-<instance part="ANT1" gate="G$1" x="60.96" y="1.27"/>
+<instance part="ANT1" gate="G$1" x="55.88" y="2.54"/>
 </instances>
 <busses>
@@
 <pinref part="B1" gate="G$1" pin="GND/DC"/>
 <wire x1="66.04" y1="-25.4" x2="67.31" y2="-25.4" width="0.1524" layer="91"/>
+<junction x="73.66" y="-29.21"/>
 </segment>
 <segment>
 <pinref part="GND15" gate="G$1" pin="GND"/>
-<wire x1="55.88" y1="-5.08" x2="55.88" y2="-3.81" width="0.1524" layer="91"/>
+<wire x1="50.8" y1="-3.81" x2="50.8" y2="-2.54" width="0.1524" layer="91"/>
 <pinref part="ANT1" gate="G$1" pin="GND"/>
 </segment>
@@
 </segment>
 </net>
-<net name="N$5" class="0">
-<segment>
-<pinref part="B1" gate="G$1" pin="B1"/>
-<pinref part="C18" gate="G$1" pin="2"/>
-<wire x1="81.28" y1="-5.08" x2="80.01" y2="-5.08" width="0.1524" layer="91"/>
-</segment>
-</net>
-<net name="N$6" class="0">
-<segment>
-<pinref part="B1" gate="G$1" pin="B2"/>
-<pinref part="C19" gate="G$1" pin="2"/>
-<wire x1="81.28" y1="-25.4" x2="80.01" y2="-25.4" width="0.1524" layer="91"/>
-</segment>
-</net>
 <net name="RFP" class="0">
 <segment>
@@
 </segment>
 <segment>
-<pinref part="C19" gate="G$1" pin="1"/>
-<wire x1="88.9" y1="-25.4" x2="90.17" y2="-25.4" width="0.1524" layer="91"/>
-<label x="90.17" y="-25.4" size="1.27" layer="95" xref="yes"/>
+<pinref part="B1" gate="G$1" pin="B2"/>
+<wire x1="80.01" y1="-25.4" x2="81.28" y2="-25.4" width="0.1524" layer="91"/>
+<label x="81.28" y="-25.4" size="1.27" layer="95" xref="yes"/>
 </segment>
 </net>
@@
 </segment>
 <segment>
-<pinref part="C18" gate="G$1" pin="1"/>
-<wire x1="88.9" y1="-5.08" x2="90.17" y2="-5.08" width="0.1524" layer="91"/>
-<label x="90.17" y="-5.08" size="1.27" layer="95" xref="yes"/>
+<pinref part="B1" gate="G$1" pin="B1"/>
+<wire x1="81.28" y1="-5.08" x2="80.01" y2="-5.08" width="0.1524" layer="91"/>
+<label x="81.28" y="-5.08" size="1.27" layer="95" xref="yes"/>
 </segment>
 </net>
@@
 </segment>
 </net>
-<net name="N$4" class="0">
+<net name="ANT" class="0">
+<segment>
+<pinref part="ANT1" gate="G$1" pin="ANT"/>
+<wire x1="55.88" y1="-2.54" x2="55.88" y2="-5.08" width="0.1524" layer="91"/>
+<pinref part="C19" gate="G$1" pin="2"/>
+<wire x1="55.88" y1="-5.08" x2="58.42" y2="-5.08" width="0.1524" layer="91"/>
+</segment>
+</net>
+<net name="N$5" class="0">
 <segment>
 <pinref part="B1" gate="G$1" pin="UN"/>
-<wire x1="67.31" y1="-5.08" x2="60.96" y2="-5.08" width="0.1524" layer="91"/>
-<wire x1="60.96" y1="-5.08" x2="60.96" y2="-3.81" width="0.1524" layer="91"/>
-<pinref part="ANT1" gate="G$1" pin="ANT"/>
-</segment>
-</net>
+<pinref part="C19" gate="G$1" pin="1"/>
+<wire x1="66.04" y1="-5.08" x2="67.31" y2="-5.08" width="0.1524" layer="91"/>
+</segment>
+</net>

Commit message: 1st revision board is done
Parts:
- removed R4: 0, jack:R-EU
- removed U$3: JACK-LOGO, jack:JACK-LOGO
- added LOGO1: HACK-LOGO, hack:HACK-LOGO
Connections:
- removed net AGND: C1.2, C14.2, C6.-, IC4ATSAMR21G-PWR-ANA.GNDANA@1, IC4ATSAMR21G-PWR-ANA.GNDANA@2, IC4ATSAMR21G-PWR-ANA.GNDANA@3, IC4ATSAMR21G-PWR-ANA.GNDANA@4, JP5.1, R4.2
- net GND: now also C1.2, C14.2, C6.-, IC4ATSAMR21G-PWR-ANA.GNDANA@1, IC4ATSAMR21G-PWR-ANA.GNDANA@2, IC4ATSAMR21G-PWR-ANA.GNDANA@3, IC4ATSAMR21G-PWR-ANA.GNDANA@4, JP5.1; no longer R4.1
Other:
- note added: "Created by Michele Perla 2015 https://hackaday.io/project/8007-hack"
- note added: "PCB Antenna and balun"
- note removed: "Created by Michele Perla 2015 https://hackaday.io/project/6062-jack"
- moved on the sheet: C19, JP1, JP5, JP6
