File: hack.sch (EAGLE design)
At the start: 42 parts, among them IC1 NUF2221W1T2G, IC3 LDO, IC4 ATSAMR21G, J1 USB-micro, SW1 SPST3.5X6MM, X1 TSX-3225 16 MHz, X2 MC-306 32.768 KHz

Commit message: 3D model added
It's missing the balun and the 32.768 KHz crystal models only
Parts:
- JP5: EAGLEUP (none) -> 1x5_FEMALE
Changed lines of the file:
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@@
 <setting verticaltext="up"/>
 </settings>
-<grid distance="0.05" unitdist="inch" unit="inch" style="lines" multiple="1" display="no" altdistance="0.01" altunitdist="inch" altunit="inch"/>
+<grid distance="0.1" unitdist="inch" unit="inch" style="lines" multiple="1" display="no" altdistance="0.01" altunitdist="inch" altunit="inch"/>
 <layers>
 <layer number="1" name="Top" color="4" fill="1" visible="no" active="no"/>
@@
 <part name="GND14" library="cortexm0" deviceset="GND" device=""/>
 <part name="GND15" library="cortexm0" deviceset="GND" device=""/>
-<part name="JP5" library="pinhead" deviceset="PINHD-1X5" device=""/>
+<part name="JP5" library="pinhead" deviceset="PINHD-1X5" device="">
+<attribute name="EAGLEUP" value="1x5_FEMALE"/>
+</part>
 <part name="JP6" library="pinhead" deviceset="PINHD-1X10" device=""/>
 <part name="ANT1" library="hack" deviceset="PCB-ANTENNA" device=""/>
@@
 <instance part="GND14" gate="G$1" x="77.47" y="-35.56"/>
 <instance part="GND15" gate="G$1" x="54.61" y="-8.89"/>
-<instance part="JP5" gate="A" x="133.35" y="0" rot="MR0"/>
+<instance part="JP5" gate="A" x="133.35" y="0" rot="MR0">
+<attribute name="EAGLEUP" x="133.35" y="0" size="1.778" layer="96" rot="MR0" display="off"/>
+</instance>
 <instance part="JP6" gate="A" x="133.35" y="-22.86" rot="MR0"/>
 <instance part="ANT1" gate="G$1" x="59.69" y="-2.54"/>

Commit message: Migrating project to KiCAD
Parts:
- removed ANT1: PCB-ANTENNA, hack:PCB-ANTENNA
- removed B1: BALUN, hack:BALUN
- removed C12, C13: 15pF, jack:C-EU
- removed C14, C15, C2, C5: 100nF, jack:C-EU
- removed C19: 22pF, jack:C-EU
- removed D1, D2: BAT60J, diode:BAT60J
- removed IC4: ATSAMR21G, hack:ATSAMR21G
- removed JP1: (no value), pinhead:PINHD-1X17
- removed JP5: (no value), pinhead:PINHD-1X5
- removed JP6: (no value), pinhead:PINHD-1X10
- removed X1: TSX-3225 16 MHz, jack:XTALCX-3225
- added JP2, JP3: (no value), pinhead:PINHD-1X14
- added U1: ATSAMD21E, hack:ATSAMD21E
- IC3: device jack:LDO -> hack:LDO
Connections:
- removed net ANT: ANT1.ANT, C19.2
- removed net AVDD: C14.1, IC4ATSAMR21G-PWR-ANA.AVDD
- removed net LDOIN: C10.+, D1.C, D2.C, IC3.VIN
- removed net N$5: B1.UN, C19.1
- removed net PA12: IC4ATSAMR21G.PA12/D, JP6.1
- removed net PA13: IC4ATSAMR21G.PA13/D, JP6.2
- removed net PB02: IC4ATSAMR21G.PB02/A, JP1.5
- removed net PB03: IC4ATSAMR21G.PB03/A, JP1.4
- removed net PB22: IC4ATSAMR21G.PB22/D, JP1.12
- removed net PB23: IC4ATSAMR21G.PB23/D, JP1.11
- removed net RFN: B1.B1, IC4ATSAMR21G.RFN
- removed net RFP: B1.B2, IC4ATSAMR21G.RFP
- removed net XTAL1: C12.1, IC4ATSAMR21G.XTAL1, X1.P$1
- removed net XTAL2: C13.1, IC4ATSAMR21G.XTAL2, X1.P$3
- new net PA02: JP3.1, U1.PA02/A
- new net PA03: JP3.2, U1.PA03/A
- new net PA10: JP3.11, U1.PA10/D
- new net PA11: JP3.12, U1.PA11/D
- net !RESET: now also JP2.11, U1.!RESET; no longer IC4ATSAMR21G.!RESET, JP1.9
- net D+OUT: now also U1.PA25/USB-DP; no longer IC4ATSAMR21G.PA25/D/USB_DP
- net D-OUT: now also U1.PA24/USB-DM; no longer IC4ATSAMR21G.PA24/D/USB_DM
- net GND: now also JP2.2, JP3.8, U1.GND, U1.GNDANA, X2.GND@1, X2.GND@2; no longer ANT1.GND, B1.GND, B1.GND/DC, B1.P$1, C12.2, C13.2, C14.2, C15.2, C2.2, C5.2, IC4ATSAMR121G-PWR-IO-1.GND, IC4ATSAMR21G-PWR-ANA.GNDANA@1, IC4ATSAMR21G-PWR-ANA.GNDANA@2, IC4ATSAMR21G-PWR-ANA.GNDANA@3, IC4ATSAMR21G-PWR-ANA.GNDANA@4, IC4ATSAMR21G-PWR-D.GND, IC4ATSAMR21G-PWR-D.PAD, IC4ATSAMR21G-PWR-IN-CORE.GND, IC4ATSAMR21G-PWR-IO-2.GND, JP1.16, JP5.1, X1.GND@1, X1.GND@2
- net N$2: now also U1.VDDCORE; no longer IC4ATSAMR21G-PWR-IN-CORE.VDDCORE
- net PA04: now also JP3.3, U1.PA04/A; no longer IC4ATSAMR21G.PA04/A, JP1.3
- net PA05: now also JP3.4, U1.PA05/A; no longer IC4ATSAMR21G.PA05/A, JP1.2
- net PA06: now also JP3.5, U1.PA06/A; no longer IC4ATSAMR21G.PA06/A, JP1.1
- net PA07: now also JP3.6, U1.PA07/A; no longer IC4ATSAMR21G.PA07/A, JP5.3
- net PA08: now also JP3.9, U1.PA08/D; no longer IC4ATSAMR21G.PA08/D, JP5.4
- net PA09: now also JP3.10, U1.PA09/D; no longer IC4ATSAMR21G.PA09/D, JP5.5
- net PA14: now also JP3.13, U1.PA14/XIN; no longer IC4ATSAMR21G.PA14/D/XIN, JP6.3
- net PA15: now also JP3.14, U1.PA15/XOUT; no longer IC4ATSAMR21G.PA15/D/XOUT, JP6.4
- net PA16: now also JP2.4, U1.PA16/D; no longer IC4ATSAMR21G.PA16/D, JP6.5
- net PA17: now also JP2.5, U1.PA17/D; no longer IC4ATSAMR21G.PA17/D, JP6.6
- net PA18: now also JP2.6, U1.PA18/D; no longer IC4ATSAMR21G.PA18/D, JP6.7
- net PA19: now also JP2.7, U1.PA19/D; no longer IC4ATSAMR21G.PA19/D, JP6.8
- net PA22: now also JP2.8, U1.PA22/D; no longer IC4ATSAMR21G.PA22/D, JP6.9
- net PA23: now also JP2.9, U1.PA23/D/USB-SOF; no longer IC4ATSAMR21G.PA23/D, JP6.10
- net PA27: now also JP2.10, U1.PA27/D; no longer IC4ATSAMR21G.PA27/D, JP1.10
- net PA28: now also JP2.12, U1.PA28/D; no longer IC4ATSAMR21G.PA28/D, JP1.8
- net SWCLK: now also JP2.13, U1.PA30/D/SWCLK; no longer IC4ATSAMR21G.PA30/SWCLK, JP1.7
- net SWDIO: now also JP2.14, U1.PA31/D/SWDIO; no longer IC4ATSAMR21G.PA31/SWDIO, JP1.6
- net VBUS: now also JP2.1; no longer D1.A, J1.VBUS, JP1.17
- net VDD: no longer JP1.14
- net VDDANA: now also JP3.7, U1.VDDANA; no longer IC4ATSAMR21G-PWR-ANA.VDDANA, JP5.2
- net VDDF: now also JP2.3, U1.VDDIN; no longer C15.1, C2.1, C5.1, IC4ATSAMR121G-PWR-IO-1.VDDIO, IC4ATSAMR21G-PWR-D.DVDD, IC4ATSAMR21G-PWR-IN-CORE.VDDIN, IC4ATSAMR21G-PWR-IO-2.VDDIO, JP1.13
- net VIN: now also C10.+, IC3.VIN, J1.VBUS; no longer D2.A, JP1.15
- net XIN32: now also U1.PA00/XIN32; no longer IC4ATSAMR21G.PA00/XIN32
- net XOUT32: now also U1.PA01/XOUT32; no longer IC4ATSAMR21G.PA01/XOUT32
Other:
- note added: "Place near ground star point"
- moved on the sheet: C1, C3, C4, C6, L1
