File: hack.brd (EAGLE design)
At the start: 44.5 x 31.9 mm, 42 parts, among them IC1 NUF2221W1T2G, IC3 LDO, IC4 ATSAMR21G, J1 USB-micro, SW1 SPST3.5X6MM, X1 TSX-3225 16 MHz, X2 MC-306 32.768 KHz

Commit message: Migrating project to KiCAD
Parts:
- removed ANT1: PCB-ANTENNA, hack:PCB-ANTENNA
- removed B1: BALUN, hack:BALUN
- removed C12, C13: 15pF, jack:C0402
- removed C14, C15, C2, C5: 100nF, jack:C0402
- removed C19: 22pF, jack:C0402
- removed D1, D2: BAT60J, diode:SOD323_ST
- removed IC4: ATSAMR21G, hack:QFN48-PAD
- removed JP1: (no value), pinhead:1X17
- removed JP5: (no value), pinhead:1X05
- removed JP6: (no value), pinhead:1X10
- removed X1: TSX-3225 16 MHz, jack:CX-3225
- added JP2, JP3: (no value), pinhead:1X14
- added U1: ATSAMD21E, hack:TQFP32
- IC3: device jack:SOT-223-3 -> hack:SOT-223-3
- moved R2 34.5 mm to (39.1, 11.4), turned to 90 degrees
- moved SW1 32.4 mm to (42.1, 18.2), turned to 270 degrees
- moved R3 29.5 mm to (37.4, 11.4), turned to 90 degrees
- moved R5 27.0 mm to (23.3, 5.25)
- moved L1 21.1 mm to (19.7, 21.1), turned to 45 degrees
- moved LOGO1 20.6 mm to (38.4, 5.25)
- moved C6 17.8 mm to (20.9, 19.9), turned to 225 degrees
- moved C1 15.4 mm to (22.1, 18.8), turned to 225 degrees
- moved D3 13.3 mm to (14.6, 14.7), turned to 90 degrees
- moved X2 9.83 mm to (32.9, 18.1), turned to 45 degrees
- moved C17 9.65 mm to (30.9, 19.4), turned to 45 degrees
- moved C11 9.65 mm to (10.2, 12.8), turned to 0 degrees
- moved U$6 9.63 mm to (40.0, 10.3)
- moved C16 9.46 mm to (34.2, 16.1), turned to 45 degrees
- moved U$5 9.43 mm to (40.0, 15.0)
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Connections:
- removed net ANT: ANT1.ANT, C19.2
- removed net AVDD: C14.1, IC4.7
- removed net LDOIN: C10.+, D1.C, D2.C, IC3.3
- removed net N$5: B1.1, C19.1
- removed net PA12: IC4.21, JP6.1
- removed net PA13: IC4.22, JP6.2
- removed net PB02: IC4.47, JP1.5
- removed net PB03: IC4.48, JP1.4
- removed net PB22: IC4.37, JP1.12
- removed net PB23: IC4.38, JP1.11
- removed net RFN: B1.3, IC4.19
- removed net RFP: B1.4, IC4.18
- removed net XTAL1: C12.1, IC4.4, X1.1
- removed net XTAL2: C13.1, IC4.3, X1.3
- new net PA02: JP3.1, U1.3
- new net PA03: JP3.2, U1.4
- new net PA10: JP3.11, U1.13
- new net PA11: JP3.12, U1.14
- net !RESET: now also JP2.11, U1.26; no longer IC4.40, JP1.9
- net D+OUT: now also U1.24; no longer IC4.34
- net D-OUT: now also U1.23; no longer IC4.33
- net GND: now also JP2.2, JP3.8, U1.10, U1.28, X2.2, X2.3; no longer ANT1.GND, B1.2, B1.5, B1.6, C12.2, C13.2, C14.2, C15.2, C2.2, C5.2, IC4.14, IC4.17, IC4.20, IC4.29, IC4.35, IC4.42, IC4.49, IC4.5, IC4.8, JP1.16, JP5.1, X1.2, X1.4
- net N$2: now also U1.29; no longer IC4.43
- net PA04: now also JP3.3, U1.5; no longer IC4.9, JP1.3
- net PA05: now also JP3.4, U1.6; no longer IC4.10, JP1.2
- net PA06: now also JP3.5, U1.7; no longer IC4.11, JP1.1
- net PA07: now also JP3.6, U1.8; no longer IC4.12, JP5.3
- net PA08: now also JP3.9, U1.11; no longer IC4.15, JP5.4
- net PA09: now also JP3.10, U1.12; no longer IC4.16, JP5.5
- net PA14: now also JP3.13, U1.15; no longer IC4.23, JP6.3
- net PA15: now also JP3.14, U1.16; no longer IC4.24, JP6.4
- net PA16: now also JP2.4, U1.17; no longer IC4.25, JP6.5
- net PA17: now also JP2.5, U1.18; no longer IC4.26, JP6.6
- net PA18: now also JP2.6, U1.19; no longer IC4.27, JP6.7
- net PA19: now also JP2.7, U1.20; no longer IC4.28, JP6.8
- net PA22: now also JP2.8, U1.21; no longer IC4.31, JP6.9
- net PA23: now also JP2.9, U1.22; no longer IC4.32, JP6.10
- net PA27: now also JP2.10, U1.25; no longer IC4.39, JP1.10
- net PA28: now also JP2.12, U1.27; no longer IC4.41, JP1.8
- net SWCLK: now also JP2.13, U1.31; no longer IC4.45, JP1.7
- net SWDIO: now also JP2.14, U1.32; no longer IC4.46, JP1.6
- net VBUS: now also JP2.1; no longer D1.A, J1.1, JP1.17
- net VDD: no longer JP1.14
- net VDDANA: now also JP3.7, U1.9; no longer IC4.6, JP5.2
- net VDDF: now also JP2.3, U1.30; no longer C15.1, C2.1, C5.1, IC4.13, IC4.30, IC4.36, IC4.44, JP1.13
- net VIN: now also C10.+, IC3.3, J1.1; no longer D2.A, JP1.15
- net XIN32: now also U1.1; no longer IC4.1
- net XOUT32: now also U1.2; no longer IC4.2
Routing:
- net GND: track 69.3 -> 0.00 mm, vias 93 -> 0
- net VDDF: track 57.5 -> 3.12 mm, vias 6 -> 0
- net VDD: track 52.2 -> 2.16 mm, vias 2 -> 0
- net !RESET: track 34.0 -> 2.75 mm, vias 1 -> 0
- net PA06: track 26.8 -> 0.00 mm, vias 2 -> 0
- net PA05: track 24.7 -> 0.00 mm, vias 2 -> 0
- net PA23: track 24.4 -> 0.00 mm
- net VBUS: track 24.4 -> 0.00 mm, vias 2 -> 0
- net PA04: track 22.7 -> 0.00 mm, vias 2 -> 0
- net PA22: track 21.2 -> 0.00 mm
- net PA09: track 19.8 -> 0.00 mm
- net PA19: track 18.4 -> 0.00 mm
- net PA08: track 18.1 -> 0.00 mm
- net PA18: track 16.7 -> 0.00 mm
- net VDDANA: track 15.8 -> 0.00 mm
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- removed copper zone on layer 1, net ANT
- removed copper zone on layer 1, net GND
- removed copper zone on layer 1, net LDOIN
- removed copper zone on layer 1, net N$5
- removed copper zone on layer 1, net RFN
- removed copper zone on layer 1, net RFP
- removed copper zone on layer 1, net VDD
- removed copper zone on layer 1, net VDDF
Other:
- board size 44.5 x 31.9 mm -> 44.5 x 26.9 mm
