File: kicad/hack.sch (KiCad schematic (older format))
At the start: 34 parts, among them P1 USB_micro, P2 CONN_01X13, P3 CONN_01X13, P4 CONN_01X01, U1 MIC5528, U2 STF202, U3 ATSAMD21E, X1 ABS07

Commit message: Added pin header datasheet+manf# (15 pins instead of 13 because 15 is cheaper)
Parts:
- P2: manf# (none) -> 320020128
Changed lines of the file:
@@
 F 1 "CONN_01X13" V 1875 6175 40  0000 C CNB
 F 2 "hack-footprints:Pin_Castellated_1x13" H 1775 6175 40  0001 C CNB
-F 3 "" H 1775 6175 40  0000 C CNB
+F 3 "https://github.com/MickMad/HACK/tree/master/kicad/datasheets/320020128.pdf" H 1775 6175 40  0001 C CNB
+F 4 "320020128" H 1775 6175 60  0001 C CNN "manf#"
 	1    1775 6175
 	1    0    0    -1
