File: kicad/hack.sch (KiCad schematic (older format))
At the start: 34 parts, among them P1 USB_micro, P2 CONN_01X13, P3 CONN_01X13, P4 CONN_01X01, U1 MIC5528, U2 STF202, U3 ATSAMD21E, X1 ABS07

Commit message: Updated Seeedstudio cost information
Parts:
- C1, C10, C11, C2, C5, C6, C7, C8, C9, P2, P3, R1, R2, R3, R4, S1: Mfr. Part # 0 -> (none)
- P1: Mfr. Part # 0 -> (none); kicost:Seeedstudio:pricing 10:$3 -> (none)
- X1: Mfr. Part # 0 -> (none); kicost:Seeedstudio:pricing 5:$1.75 -> (none)
Changed lines of the file:
@@
 F 2 "hack-footprints:R_0603_HandSoldering" H 2025 1975 40  0001 C CNB
 F 3 "https://github.com/MickMad/HACK/tree/master/kicad/datasheets/301010151.pdf" H 2025 1975 40  0001 C CNB
-F 4 "0" H 2025 1975 60  0001 C CNN "Mfr. Part #"
-F 5 "301010151" H 2025 1975 60  0001 C CNN "manf#"
-F 6 "100:$1" H 2025 1975 60  0001 C CNN "kicost:Seeedstudio:pricing"
+F 4 "301010151" H 2025 1975 60  0001 C CNN "manf#"
+F 5 "100:$1" H 2025 1975 60  0001 C CNN "kicost:Seeedstudio:pricing"
 	1    2025 1975
 	1    0    0    -1
@@
 F 2 "hack-footprints:C_0603_HandSoldering" H 1700 1975 40  0001 C CNB
 F 3 "https://github.com/MickMad/HACK/tree/master/kicad/datasheets/0100850P1.pdf" H 1700 1975 40  0001 C CNB
-F 4 "0" H 1700 1975 60  0001 C CNN "Mfr. Part #"
-F 5 "302010144" H 1700 1975 60  0001 C CNN "manf#"
-F 6 "100:$1" H 1700 1975 60  0001 C CNN "kicost:Seeedstudio:pricing"
+F 4 "302010144" H 1700 1975 60  0001 C CNN "manf#"
+F 5 "100:$1" H 1700 1975 60  0001 C CNN "kicost:Seeedstudio:pricing"
 	1    1700 1975
 	1    0    0    -1
@@
 F 2 "hack-footprints:C_0603_HandSoldering" H 1500 4350 40  0001 C CNB
 F 3 "https://github.com/MickMad/HACK/tree/master/kicad/datasheets/302010097.pdf" H 1500 4350 40  0001 C CNB
-F 4 "0" H 1500 4350 60  0001 C CNN "Mfr. Part #"
-F 5 "302010097" H 1500 4350 60  0001 C CNN "manf#"
-F 6 "100:$1" H 1500 4350 60  0001 C CNN "kicost:Seeedstudio:pricing"
+F 4 "302010097" H 1500 4350 60  0001 C CNN "manf#"
+F 5 "100:$1" H 1500 4350 60  0001 C CNN "kicost:Seeedstudio:pricing"
 	1    1500 4350
 	1    0    0    -1
@@
 F 2 "hack-footprints:C_0603_HandSoldering" H 5300 2425 40  0001 C CNB
 F 3 "https://github.com/MickMad/HACK/tree/master/kicad/datasheets/0100020P1.pdf" H 5300 2425 40  0001 C CNB
-F 4 "0" H 5300 2425 60  0001 C CNN "Mfr. Part #"
-F 5 "302010138" H 5300 2425 60  0001 C CNN "manf#"
-F 6 "100:$2" H 5300 2425 60  0001 C CNN "kicost:Seeedstudio:pricing"
+F 4 "302010138" H 5300 2425 60  0001 C CNN "manf#"
+F 5 "100:$2" H 5300 2425 60  0001 C CNN "kicost:Seeedstudio:pricing"
 	1    5300 2425
 	-1   0    0    -1
@@
 F 2 "hack-footprints:Pin_Castellated_1x13" H 1775 6175 40  0001 C CNB
 F 3 "https://github.com/MickMad/HACK/tree/master/kicad/datasheets/320020128.pdf" H 1775 6175 40  0001 C CNB
-F 4 "0" H 1775 6175 60  0001 C CNN "Mfr. Part #"
-F 5 "320020128" H 1775 6175 60  0001 C CNN "manf#"
-F 6 "30:$2.4" H 1775 6175 60  0001 C CNN "kicost:Seeedstudio:pricing"
+F 4 "320020128" H 1775 6175 60  0001 C CNN "manf#"
+F 5 "30:$2.4" H 1775 6175 60  0001 C CNN "kicost:Seeedstudio:pricing"
 	1    1775 6175
 	1    0    0    -1
@@
 F 2 "hack-footprints:R_0603_HandSoldering" H 8050 2625 40  0001 C CNB
 F 3 "https://github.com/MickMad/HACK/tree/master/kicad/datasheets/0011330P1.pdf" H 8050 2625 40  0001 C CNB
-F 4 "0" H 8050 2625 60  0001 C CNN "Mfr. Part #"
-F 5 "301010300" H 8050 2625 60  0001 C CNN "manf#"
-F 6 "100:$1" H 8050 2625 60  0001 C CNN "kicost:Seeedstudio:pricing"
+F 4 "301010300" H 8050 2625 60  0001 C CNN "manf#"
+F 5 "100:$1" H 8050 2625 60  0001 C CNN "kicost:Seeedstudio:pricing"
 	1    8050 2625
 	1    0    0    -1
@@
 F 2 "hack-footprints:SPST-PTS_810" H 9350 2950 40  0001 C CNB
 F 3 "https://github.com/MickMad/HACK/tree/master/kicad/datasheets/311020045.pdf" H 9350 2950 40  0001 C CNB
-F 4 "0" H 9350 2950 60  0001 C CNN "Mfr. Part #"
-F 5 "311020045" V 9350 2950 60  0001 C CNN "manf#"
-F 6 "10:$2.036" V 9350 2950 60  0001 C CNN "kicost:Seeedstudio:pricing"
+F 4 "311020045" V 9350 2950 60  0001 C CNN "manf#"
+F 5 "10:$2.036" V 9350 2950 60  0001 C CNN "kicost:Seeedstudio:pricing"
 	1    9350 2950
 	0    1    -1   0
@@
 F 2 "hack-footprints:R_0603_HandSoldering" H 8975 2175 40  0001 C CNB
 F 3 "https://github.com/MickMad/HACK/tree/master/kicad/datasheets/0011240P1.pdf" H 8975 2175 40  0001 C CNB
-F 4 "0" H 8975 2175 60  0001 C CNN "Mfr. Part #"
-F 5 "301010299" H 8975 2175 60  0001 C CNN "manf#"
-F 6 "100:$1" H 8975 2175 60  0001 C CNN "kicost:Seeedstudio:pricing"
+F 4 "301010299" H 8975 2175 60  0001 C CNN "manf#"
+F 5 "100:$1" H 8975 2175 60  0001 C CNN "kicost:Seeedstudio:pricing"
 	1    8975 2175
 	1    0    0    1
@@
 F 2 "hack-footprints:C_0603_HandSoldering" H 1500 3350 40  0001 C CNB
 F 3 "https://github.com/MickMad/HACK/tree/master/kicad/datasheets/UPY-GPHC_X5R_4V-to-50V_14_0717-202131.pdf" H 1500 3350 40  0001 C CNB
-F 4 "0" H 1500 3350 60  0001 C CNN "Mfr. Part #"
-F 5 "CC0603MRX5R5BB225" H 1500 3350 60  0001 C CNN "manf#"
+F 4 "CC0603MRX5R5BB225" H 1500 3350 60  0001 C CNN "manf#"
 	1    1500 3350
 	1    0    0    -1
@@
 F 2 "hack-footprints:ST-USB-001G" H 1250 1150 60  0001 C CNN
 F 3 "https://github.com/MickMad/HACK/tree/master/kicad/datasheets/320010000.pdf" H 1250 1200 60  0001 C CNN
-F 4 "0" H 1250 1150 60  0001 C CNN "Mfr. Part #"
-F 5 "320010000" H 1350 1300 60  0001 C CNN "manf#"
-F 6 "10:$3" H 1250 1150 60  0001 C CNN "kicost:Seeedstudio:pricing"
+F 4 "320010000" H 1350 1300 60  0001 C CNN "manf#"
 	1    1250 1150
 	1    0    0    -1
@@
 F 2 "hack-footprints:C_0603_HandSoldering" H 2800 3350 40  0001 C CNB
 F 3 "https://github.com/MickMad/HACK/tree/master/kicad/datasheets/UPY-GPHC_X5R_4V-to-50V_14_0717-202131.pdf" H 2800 3350 40  0001 C CNB
-F 4 "0" H 2800 3350 60  0001 C CNN "Mfr. Part #"
-F 5 "CC0603MRX5R5BB225" H 2800 3350 60  0001 C CNN "manf#"
+F 4 "CC0603MRX5R5BB225" H 2800 3350 60  0001 C CNN "manf#"
 	1    2800 3350
 	1    0    0    -1
@@
 F 2 "hack-footprints:C_0603_HandSoldering" H 2700 4350 40  0001 C CNB
 F 3 "https://github.com/MickMad/HACK/tree/master/kicad/datasheets/302010097.pdf" H 2700 4350 40  0001 C CNB
-F 4 "0" H 2700 4350 60  0001 C CNN "Mfr. Part #"
-F 5 "302010097" H 2700 4350 60  0001 C CNN "manf#"
-F 6 "100:$1" H 2700 4350 60  0001 C CNN "kicost:Seeedstudio:pricing"
+F 4 "302010097" H 2700 4350 60  0001 C CNN "manf#"
+F 5 "100:$1" H 2700 4350 60  0001 C CNN "kicost:Seeedstudio:pricing"
 	1    2700 4350
 	1    0    0    -1
@@
 F 2 "hack-footprints:xtal_3.2x1.5mm" H 2100 4050 60  0001 C CNN
 F 3 "https://github.com/MickMad/HACK/tree/master/kicad/datasheets/306010055.pdf" H 2100 3900 60  0001 C CNN
-F 4 "0" H 2100 4050 60  0001 C CNN "Mfr. Part #"
-F 5 "306010055" H 2200 4000 60  0001 C CNN "manf#"
-F 6 "5:$1.75" H 2100 4050 60  0001 C CNN "kicost:Seeedstudio:pricing"
+F 4 "306010055" H 2200 4000 60  0001 C CNN "manf#"
 	1    2100 4050
 	1    0    0    -1
@@
 F 2 "hack-footprints:Pin_Castellated_1x13" H 2625 6175 40  0001 C CNB
 F 3 "https://github.com/MickMad/HACK/tree/master/kicad/datasheets/320020128.pdf" H 2625 6175 40  0001 C CNB
-F 4 "0" H 2625 6175 60  0001 C CNN "Mfr. Part #"
-F 5 "320020128" H 2625 6175 60  0001 C CNN "manf#"
-F 6 "30:$2.4" H 2625 6175 60  0001 C CNN "kicost:Seeedstudio:pricing"
+F 4 "320020128" H 2625 6175 60  0001 C CNN "manf#"
+F 5 "30:$2.4" H 2625 6175 60  0001 C CNN "kicost:Seeedstudio:pricing"
 	1    2625 6175
 	-1   0    0    1
@@
 F 2 "hack-footprints:R_0603_HandSoldering" H 9350 2625 40  0001 C CNB
 F 3 "https://github.com/MickMad/HACK/tree/master/kicad/datasheets/0011330P1.pdf" H 9350 2625 40  0001 C CNB
-F 4 "0" H 9350 2625 60  0001 C CNN "Mfr. Part #"
-F 5 "301010300" H 9350 2625 60  0001 C CNN "manf#"
-F 6 "100:$1" H 9350 2625 60  0001 C CNN "kicost:Seeedstudio:pricing"
+F 4 "301010300" H 9350 2625 60  0001 C CNN "manf#"
+F 5 "100:$1" H 9350 2625 60  0001 C CNN "kicost:Seeedstudio:pricing"
 	1    9350 2625
 	1    0    0    -1
@@
 F 2 "hack-footprints:C_0603_HandSoldering" H 7550 2025 40  0001 C CNB
 F 3 "https://github.com/MickMad/HACK/tree/master/kicad/datasheets/0100020P1.pdf" H 7550 2025 40  0001 C CNB
-F 4 "0" H 7550 2025 60  0001 C CNN "Mfr. Part #"
-F 5 "302010138" H 7550 2025 60  0001 C CNN "manf#"
-F 6 "100:$2" H 7550 2025 60  0001 C CNN "kicost:Seeedstudio:pricing"
+F 4 "302010138" H 7550 2025 60  0001 C CNN "manf#"
+F 5 "100:$2" H 7550 2025 60  0001 C CNN "kicost:Seeedstudio:pricing"
 	1    7550 2025
 	-1   0    0    -1
@@
 F 2 "hack-footprints:C_0603_HandSoldering" H 8050 2025 40  0001 C CNB
 F 3 "https://github.com/MickMad/HACK/tree/master/kicad/datasheets/0100020P1.pdf" H 8050 2025 40  0001 C CNB
-F 4 "0" H 8050 2025 60  0001 C CNN "Mfr. Part #"
-F 5 "302010138" H 8050 2025 60  0001 C CNN "manf#"
-F 6 "100:$2" H 8050 2025 60  0001 C CNN "kicost:Seeedstudio:pricing"
+F 4 "302010138" H 8050 2025 60  0001 C CNN "manf#"
+F 5 "100:$2" H 8050 2025 60  0001 C CNN "kicost:Seeedstudio:pricing"
 	1    8050 2025
 	-1   0    0    -1
@@
 F 2 "hack-footprints:C_0603_HandSoldering" H 8975 2950 40  0001 C CNB
 F 3 "https://github.com/MickMad/HACK/tree/master/kicad/datasheets/0100020P1.pdf" H 8975 2950 40  0001 C CNB
-F 4 "0" H 8975 2950 60  0001 C CNN "Mfr. Part #"
-F 5 "302010138" H 8975 2950 60  0001 C CNN "manf#"
-F 6 "100:$2" H 8975 2950 60  0001 C CNN "kicost:Seeedstudio:pricing"
+F 4 "302010138" H 8975 2950 60  0001 C CNN "manf#"
+F 5 "100:$2" H 8975 2950 60  0001 C CNN "kicost:Seeedstudio:pricing"
 	1    8975 2950
 	-1   0    0    -1

Commit message: Fixed KiCost BOM issue, updated BOM
Parts:
- C10, C11, C8, C9: kicost:Seeedstudio:pricing 100:$2 -> (none); kicost:pricing (none) -> 1:$0.02
- C5, C6, R1, R2, R3, R4: kicost:Seeedstudio:pricing 100:$1 -> (none); kicost:pricing (none) -> 1:$0.01
- D1: kicost:pricing (none) -> 1:$0.03
- P2, P3: kicost:Seeedstudio:pricing 30:$2.4 -> (none); kicost:pricing (none) -> 1:$0.08
- S1: kicost:Seeedstudio:pricing 10:$2.036 -> (none); kicost:pricing (none) -> 1:$0.2036
Changed lines of the file:
@@
 F 3 "https://github.com/MickMad/HACK/tree/master/kicad/datasheets/301010151.pdf" H 2025 1975 40  0001 C CNB
 F 4 "301010151" H 2025 1975 60  0001 C CNN "manf#"
-F 5 "100:$1" H 2025 1975 60  0001 C CNN "kicost:Seeedstudio:pricing"
+F 5 "1:$0.01" H 2025 1975 60  0001 C CNN "kicost:pricing"
 	1    2025 1975
 	1    0    0    -1
@@
 F 3 "https://github.com/MickMad/HACK/tree/master/kicad/datasheets/0100850P1.pdf" H 1700 1975 40  0001 C CNB
 F 4 "302010144" H 1700 1975 60  0001 C CNN "manf#"
-F 5 "100:$1" H 1700 1975 60  0001 C CNN "kicost:Seeedstudio:pricing"
+F 5 "1:$0.01" H 1700 1975 60  0001 C CNN "kicost:pricing"
 	1    1700 1975
 	1    0    0    -1
@@
 F 3 "https://github.com/MickMad/HACK/tree/master/kicad/datasheets/302010097.pdf" H 1500 4350 40  0001 C CNB
 F 4 "302010097" H 1500 4350 60  0001 C CNN "manf#"
-F 5 "100:$1" H 1500 4350 60  0001 C CNN "kicost:Seeedstudio:pricing"
+F 5 "1:$0.01" H 1500 4350 60  0001 C CNN "kicost:pricing"
 	1    1500 4350
 	1    0    0    -1
@@
 F 3 "https://github.com/MickMad/HACK/tree/master/kicad/datasheets/0100020P1.pdf" H 5300 2425 40  0001 C CNB
 F 4 "302010138" H 5300 2425 60  0001 C CNN "manf#"
-F 5 "100:$2" H 5300 2425 60  0001 C CNN "kicost:Seeedstudio:pricing"
+F 5 "1:$0.02" H 5300 2425 60  0001 C CNN "kicost:pricing"
 	1    5300 2425
 	-1   0    0    -1
@@
 F 3 "https://github.com/MickMad/HACK/tree/master/kicad/datasheets/320020128.pdf" H 1775 6175 40  0001 C CNB
 F 4 "320020128" H 1775 6175 60  0001 C CNN "manf#"
-F 5 "30:$2.4" H 1775 6175 60  0001 C CNN "kicost:Seeedstudio:pricing"
+F 5 "1:$0.08" H 1775 6175 60  0001 C CNN "kicost:pricing"
 	1    1775 6175
 	1    0    0    -1
@@
 F 3 "https://github.com/MickMad/HACK/tree/master/kicad/datasheets/0330020P1.pdf" V 8050 2950 40  0001 C CNB
 F 4 "304090042" V 8050 2950 60  0001 C CNN "manf#"
+F 5 "1:$0.03" V 8050 2950 60  0001 C CNN "kicost:pricing"
 	1    8050 2950
 	0    -1   -1   0
@@
 F 3 "https://github.com/MickMad/HACK/tree/master/kicad/datasheets/0011330P1.pdf" H 8050 2625 40  0001 C CNB
 F 4 "301010300" H 8050 2625 60  0001 C CNN "manf#"
-F 5 "100:$1" H 8050 2625 60  0001 C CNN "kicost:Seeedstudio:pricing"
+F 5 "1:$0.01" H 8050 2625 60  0001 C CNN "kicost:pricing"
 	1    8050 2625
 	1    0    0    -1
@@
 F 3 "https://github.com/MickMad/HACK/tree/master/kicad/datasheets/311020045.pdf" H 9350 2950 40  0001 C CNB
 F 4 "311020045" V 9350 2950 60  0001 C CNN "manf#"
-F 5 "10:$2.036" V 9350 2950 60  0001 C CNN "kicost:Seeedstudio:pricing"
+F 5 "1:$0.2036" V 9350 2950 60  0001 C CNN "kicost:pricing"
 	1    9350 2950
 	0    1    -1   0
@@
 F 3 "https://github.com/MickMad/HACK/tree/master/kicad/datasheets/0011240P1.pdf" H 8975 2175 40  0001 C CNB
 F 4 "301010299" H 8975 2175 60  0001 C CNN "manf#"
-F 5 "100:$1" H 8975 2175 60  0001 C CNN "kicost:Seeedstudio:pricing"
+F 5 "1:$0.01" H 8975 2175 60  0001 C CNN "kicost:pricing"
 	1    8975 2175
 	1    0    0    1
@@
 F 3 "https://github.com/MickMad/HACK/tree/master/kicad/datasheets/320020128.pdf" H 2625 6175 40  0001 C CNB
 F 4 "320020128" H 2625 6175 60  0001 C CNN "manf#"
-F 5 "30:$2.4" H 2625 6175 60  0001 C CNN "kicost:Seeedstudio:pricing"
+F 5 "1:$0.08" H 2625 6175 60  0001 C CNN "kicost:pricing"
 	1    2625 6175
 	-1   0    0    1
@@
 F 3 "https://github.com/MickMad/HACK/tree/master/kicad/datasheets/0011330P1.pdf" H 9350 2625 40  0001 C CNB
 F 4 "301010300" H 9350 2625 60  0001 C CNN "manf#"
-F 5 "100:$1" H 9350 2625 60  0001 C CNN "kicost:Seeedstudio:pricing"
+F 5 "1:$0.01" H 9350 2625 60  0001 C CNN "kicost:pricing"
 	1    9350 2625
 	1    0    0    -1
@@
 F 3 "https://github.com/MickMad/HACK/tree/master/kicad/datasheets/0100020P1.pdf" H 7550 2025 40  0001 C CNB
 F 4 "302010138" H 7550 2025 60  0001 C CNN "manf#"
-F 5 "100:$2" H 7550 2025 60  0001 C CNN "kicost:Seeedstudio:pricing"
+F 5 "1:$0.02" H 7550 2025 60  0001 C CNN "kicost:pricing"
 	1    7550 2025
 	-1   0    0    -1
@@
 F 3 "https://github.com/MickMad/HACK/tree/master/kicad/datasheets/0100020P1.pdf" H 8050 2025 40  0001 C CNB
 F 4 "302010138" H 8050 2025 60  0001 C CNN "manf#"
-F 5 "100:$2" H 8050 2025 60  0001 C CNN "kicost:Seeedstudio:pricing"
+F 5 "1:$0.02" H 8050 2025 60  0001 C CNN "kicost:pricing"
 	1    8050 2025
 	-1   0    0    -1
@@
 F 3 "https://github.com/MickMad/HACK/tree/master/kicad/datasheets/0100020P1.pdf" H 8975 2950 40  0001 C CNB
 F 4 "302010138" H 8975 2950 60  0001 C CNN "manf#"
-F 5 "100:$2" H 8975 2950 60  0001 C CNN "kicost:Seeedstudio:pricing"
+F 5 "1:$0.02" H 8975 2950 60  0001 C CNN "kicost:pricing"
 	1    8975 2950
 	-1   0    0    -1

Commit message: Changed LED, headers, USBmicro, XTAL manf#
These parts are readily available from all distributors, previous ones
were only sold by Seeed
Parts:
- C10, C11, C8, C9: kicost:pricing 1:$0.02 -> (none); manf# 302010138 -> CC0603KRX7R9BB104
- C5: kicost:pricing 1:$0.01 -> (none); manf# 302010144 -> CC0603KRX7R9BB472
- C6: kicost:pricing 1:$0.01 -> (none); manf# 302010097 -> CC0603JRNPO9BN100
- C7: kicost:Seeedstudio:pricing 100:$1 -> (none); manf# 302010097 -> CC0603JRNPO9BN100
- D1: kicost:pricing 1:$0.03 -> (none); manf# 304090042 -> LTST-C190KRKT
- P1: manf# 320010000 -> 10118193-0001LF
- P2, P3: kicost:pricing 1:$0.08 -> (none); manf# 320020128 -> PREC014SACN-RC
- R1: kicost:pricing 1:$0.01 -> (none); manf# 301010151 -> RC0603FR-071ML
- R2, R4: kicost:pricing 1:$0.01 -> (none); manf# 301010300 -> RC0603FR-07330RL
- R3: kicost:pricing 1:$0.01 -> (none); manf# 301010299 -> RC0603FR-0710KL
- S1: kicost:pricing 1:$0.2036 -> (none); manf# 311020045 -> PTS810 SJM 250 SMTR LFS
- X1: manf# 306010055 -> ABS07-32.768KHZ-7-T
Changed lines of the file:
@@
 F 2 "hack-footprints:R_0603_HandSoldering" H 2025 1975 40  0001 C CNB
 F 3 "https://github.com/MickMad/HACK/tree/master/kicad/datasheets/301010151.pdf" H 2025 1975 40  0001 C CNB
-F 4 "301010151" H 2025 1975 60  0001 C CNN "manf#"
-F 5 "1:$0.01" H 2025 1975 60  0001 C CNN "kicost:pricing"
+F 4 "RC0603FR-071ML" H 2025 1975 60  0001 C CNN "manf#"
 	1    2025 1975
 	1    0    0    -1
@@
 F 2 "hack-footprints:C_0603_HandSoldering" H 1700 1975 40  0001 C CNB
 F 3 "https://github.com/MickMad/HACK/tree/master/kicad/datasheets/0100850P1.pdf" H 1700 1975 40  0001 C CNB
-F 4 "302010144" H 1700 1975 60  0001 C CNN "manf#"
-F 5 "1:$0.01" H 1700 1975 60  0001 C CNN "kicost:pricing"
+F 4 "CC0603KRX7R9BB472" H 1700 1975 60  0001 C CNN "manf#"
 	1    1700 1975
 	1    0    0    -1
@@
 F 2 "hack-footprints:C_0603_HandSoldering" H 1500 4350 40  0001 C CNB
 F 3 "https://github.com/MickMad/HACK/tree/master/kicad/datasheets/302010097.pdf" H 1500 4350 40  0001 C CNB
-F 4 "302010097" H 1500 4350 60  0001 C CNN "manf#"
-F 5 "1:$0.01" H 1500 4350 60  0001 C CNN "kicost:pricing"
+F 4 "CC0603JRNPO9BN100" H 1500 4350 60  0001 C CNN "manf#"
 	1    1500 4350
 	1    0    0    -1
@@
 F 2 "hack-footprints:C_0603_HandSoldering" H 5300 2425 40  0001 C CNB
 F 3 "https://github.com/MickMad/HACK/tree/master/kicad/datasheets/0100020P1.pdf" H 5300 2425 40  0001 C CNB
-F 4 "302010138" H 5300 2425 60  0001 C CNN "manf#"
-F 5 "1:$0.02" H 5300 2425 60  0001 C CNN "kicost:pricing"
+F 4 "CC0603KRX7R9BB104" H 5300 2425 60  0001 C CNN "manf#"
 	1    5300 2425
 	-1   0    0    -1
@@
 F 1 "CONN_01X13" V 1875 6175 40  0000 C CNB
 F 2 "hack-footprints:Pin_Castellated_1x13" H 1775 6175 40  0001 C CNB
-F 3 "https://github.com/MickMad/HACK/tree/master/kicad/datasheets/320020128.pdf" H 1775 6175 40  0001 C CNB
-F 4 "320020128" H 1775 6175 60  0001 C CNN "manf#"
-F 5 "1:$0.08" H 1775 6175 60  0001 C CNN "kicost:pricing"
+F 3 "https://github.com/MickMad/HACK/tree/master/kicad/datasheets/xRxCzzzSxxN-RC_ST_11635-B.pdf" H 1775 6175 40  0001 C CNB
+F 4 "PREC014SACN-RC" H 1775 6175 60  0001 C CNN "manf#"
 	1    1775 6175
 	1    0    0    -1
@@
 F 1 "RED" V 7975 2900 40  0000 R CNN
 F 2 "hack-footprints:LED_0603_HandSoldering" V 8050 2950 40  0001 C CNB
-F 3 "https://github.com/MickMad/HACK/tree/master/kicad/datasheets/0330020P1.pdf" V 8050 2950 40  0001 C CNB
-F 4 "304090042" V 8050 2950 60  0001 C CNN "manf#"
-F 5 "1:$0.03" V 8050 2950 60  0001 C CNN "kicost:pricing"
+F 3 "https://github.com/MickMad/HACK/tree/master/kicad/datasheets/S_110_LTST-C190KRKT.pdf" V 8050 2950 40  0001 C CNB
+F 4 "LTST-C190KRKT" V 8050 2950 60  0001 C CNN "manf#"
 	1    8050 2950
 	0    -1   -1   0
@@
 F 2 "hack-footprints:R_0603_HandSoldering" H 8050 2625 40  0001 C CNB
 F 3 "https://github.com/MickMad/HACK/tree/master/kicad/datasheets/0011330P1.pdf" H 8050 2625 40  0001 C CNB
-F 4 "301010300" H 8050 2625 60  0001 C CNN "manf#"
-F 5 "1:$0.01" H 8050 2625 60  0001 C CNN "kicost:pricing"
+F 4 "RC0603FR-07330RL" H 8050 2625 60  0001 C CNN "manf#"
 	1    8050 2625
 	1    0    0    -1
@@
 F 2 "hack-footprints:SPST-PTS_810" H 9350 2950 40  0001 C CNB
 F 3 "https://github.com/MickMad/HACK/tree/master/kicad/datasheets/311020045.pdf" H 9350 2950 40  0001 C CNB
-F 4 "311020045" V 9350 2950 60  0001 C CNN "manf#"
-F 5 "1:$0.2036" V 9350 2950 60  0001 C CNN "kicost:pricing"
+F 4 "PTS810 SJM 250 SMTR LFS" V 9350 2950 60  0001 C CNN "manf#"
 	1    9350 2950
 	0    1    -1   0
@@
 F 2 "hack-footprints:R_0603_HandSoldering" H 8975 2175 40  0001 C CNB
 F 3 "https://github.com/MickMad/HACK/tree/master/kicad/datasheets/0011240P1.pdf" H 8975 2175 40  0001 C CNB
-F 4 "301010299" H 8975 2175 60  0001 C CNN "manf#"
-F 5 "1:$0.01" H 8975 2175 60  0001 C CNN "kicost:pricing"
+F 4 "RC0603FR-0710KL" H 8975 2175 60  0001 C CNN "manf#"
 	1    8975 2175
 	1    0    0    1
@@
 F 1 "USB_micro" H 1250 1100 40  0000 C CNB
 F 2 "hack-footprints:ST-USB-001G" H 1250 1150 60  0001 C CNN
-F 3 "https://github.com/MickMad/HACK/tree/master/kicad/datasheets/320010000.pdf" H 1250 1200 60  0001 C CNN
-F 4 "320010000" H 1350 1300 60  0001 C CNN "manf#"
+F 3 "https://github.com/MickMad/HACK/tree/master/kicad/datasheets/10118193.pdf" H 1250 1200 60  0001 C CNN
+F 4 "10118193-0001LF" H 1350 1300 60  0001 C CNN "manf#"
 	1    1250 1150
 	1    0    0    -1
@@
 F 2 "hack-footprints:C_0603_HandSoldering" H 2700 4350 40  0001 C CNB
 F 3 "https://github.com/MickMad/HACK/tree/master/kicad/datasheets/302010097.pdf" H 2700 4350 40  0001 C CNB
-F 4 "302010097" H 2700 4350 60  0001 C CNN "manf#"
-F 5 "100:$1" H 2700 4350 60  0001 C CNN "kicost:Seeedstudio:pricing"
+F 4 "CC0603JRNPO9BN100" H 2700 4350 60  0001 C CNN "manf#"
 	1    2700 4350
 	1    0    0    -1
@@
 F 2 "hack-footprints:xtal_3.2x1.5mm" H 2100 4050 60  0001 C CNN
 F 3 "https://github.com/MickMad/HACK/tree/master/kicad/datasheets/306010055.pdf" H 2100 3900 60  0001 C CNN
-F 4 "306010055" H 2200 4000 60  0001 C CNN "manf#"
+F 4 "ABS07-32.768KHZ-7-T" H 2200 4000 60  0001 C CNN "manf#"
 	1    2100 4050
 	1    0    0    -1
@@
 F 2 "hack-footprints:Pin_Castellated_1x13" H 2625 6175 40  0001 C CNB
 F 3 "https://github.com/MickMad/HACK/tree/master/kicad/datasheets/320020128.pdf" H 2625 6175 40  0001 C CNB
-F 4 "320020128" H 2625 6175 60  0001 C CNN "manf#"
-F 5 "1:$0.08" H 2625 6175 60  0001 C CNN "kicost:pricing"
+F 4 "PREC014SACN-RC" H 2625 6175 60  0001 C CNN "manf#"
 	1    2625 6175
 	-1   0    0    1
@@
 F 2 "hack-footprints:R_0603_HandSoldering" H 9350 2625 40  0001 C CNB
 F 3 "https://github.com/MickMad/HACK/tree/master/kicad/datasheets/0011330P1.pdf" H 9350 2625 40  0001 C CNB
-F 4 "301010300" H 9350 2625 60  0001 C CNN "manf#"
-F 5 "1:$0.01" H 9350 2625 60  0001 C CNN "kicost:pricing"
+F 4 "RC0603FR-07330RL" H 9350 2625 60  0001 C CNN "manf#"
 	1    9350 2625
 	1    0    0    -1
@@
 F 2 "hack-footprints:C_0603_HandSoldering" H 7550 2025 40  0001 C CNB
 F 3 "https://github.com/MickMad/HACK/tree/master/kicad/datasheets/0100020P1.pdf" H 7550 2025 40  0001 C CNB
-F 4 "302010138" H 7550 2025 60  0001 C CNN "manf#"
-F 5 "1:$0.02" H 7550 2025 60  0001 C CNN "kicost:pricing"
+F 4 "CC0603KRX7R9BB104" H 7550 2025 60  0001 C CNN "manf#"
 	1    7550 2025
 	-1   0    0    -1
@@
 F 2 "hack-footprints:C_0603_HandSoldering" H 8050 2025 40  0001 C CNB
 F 3 "https://github.com/MickMad/HACK/tree/master/kicad/datasheets/0100020P1.pdf" H 8050 2025 40  0001 C CNB
-F 4 "302010138" H 8050 2025 60  0001 C CNN "manf#"
-F 5 "1:$0.02" H 8050 2025 60  0001 C CNN "kicost:pricing"
+F 4 "CC0603KRX7R9BB104" H 8050 2025 60  0001 C CNN "manf#"
 	1    8050 2025
 	-1   0    0    -1
@@
 F 2 "hack-footprints:C_0603_HandSoldering" H 8975 2950 40  0001 C CNB
 F 3 "https://github.com/MickMad/HACK/tree/master/kicad/datasheets/0100020P1.pdf" H 8975 2950 40  0001 C CNB
-F 4 "302010138" H 8975 2950 60  0001 C CNN "manf#"
-F 5 "1:$0.02" H 8975 2950 60  0001 C CNN "kicost:pricing"
+F 4 "CC0603KRX7R9BB104" H 8975 2950 60  0001 C CNN "manf#"
 	1    8975 2950
 	-1   0    0    -1
