File: kicad/hack.sch (KiCad schematic (older format))
At the start: 35 parts, among them P1 USB_micro, P2 CONN_01X11, P3 CONN_01X11, P4 CONN_01X06, P5 CONN_01X01, U1 MIC5528, U2 STF202, U3 ATSAMD21E, X1 ABS07

Commit message: Form factor is PDIP-24 now, ready to fab
HACK now fits a PDIP-24 package (its solderable thru-hole headers
spacing is now 0.6"); being longer there's some space on the top side,
so it now features a convenient Cortex SWD Connector, a 2x5 male pin
header with 50 mils spacing in SMD package.
Parts:
- removed FID1, FID2, FID3: FIDUCIAL, hack-footprints:FIDUCIAL, symbol FIDUCIAL
- removed P2, P3: CONN_01X11, hack-footprints:Pin_Castellated_1x11, symbol CONN_01X11
- removed P4: CONN_01X06, hack-footprints:Pin_Castellated_1x06, symbol CONN_01X06
- added P2, P3: CONN_01X14, hack-footprints:Pin_Castellated_1x14, symbol CONN_01X14
- added P5: CONN_SWD, hack-footprints:Cortex_Debug_Connector_50mils, symbol CONN_SWD
- C1, C10, C11, C2, C5, C6, C7, C8, C9: footprint hack-footprints:C_0603_HandSoldering -> hack-footprints:C_0603
- C3, C4: footprint hack-footprints:c_elec_3x5.3 -> hack-footprints:CAP_ELEC_SMD_3x5mm
- D1: footprint hack-footprints:LED_0603_HandSoldering -> hack-footprints:LED_0603
- L1: footprint hack-footprints:L_0603_HandSoldering -> hack-footprints:L_0603
- R1, R2, R3, R4: footprint hack-footprints:R_0603_HandSoldering -> hack-footprints:R_0603
- renumbered P5 to P4
Connections:
- net !RESET: now also P2.5 (P5), P5.10 (nRESET)
- net GND: now also P2.1 (P1), P3.14 (P14), P5.3 (GND), P5.5 (GND)
- net PA02/A0: now also P2.9 (P9)
- net PA03/A1: now also P2.10 (P10)
- net PA04/A2: now also P2.11 (P11)
- net PA05/A3: now also P2.12 (P12)
- net PA06/A4: now also P2.13 (P13)
- net PA07/A5: now also P2.14 (P14)
- net PA08/0: now also P3.12 (P12)
- net PA09/1: now also P3.11 (P11)
- net PA10/2: now also P3.10 (P10)
- net PA11/3: now also P3.9 (P9)
- net PA14/4: now also P3.8 (P8)
- net PA15/5: now also P3.7 (P7)
- net PA16/6: now also P3.6 (P6)
- net PA17/7: now also P3.5 (P5)
- net PA18/8: now also P3.4 (P4)
- net PA19/9: now also P3.3 (P3)
- net PA22/10: now also P3.2 (P2)
- net PA23/11: now also P3.1 (P1)
- net PA27/12: now also P2.4 (P4)
- net PA28/13: now also P2.6 (P6)
- net PA30/SWCLK: now also P2.7 (P7), P5.4 (SWDCLK)
- net PA31/SWDIO: now also P2.8 (P8), P5.2 (SWDIO)
- net VDDANA: now also P3.13 (P13)
- net VDDF: now also P2.3 (P3), P5.1 (VTref)
- net VLDO: now also P2.2 (P2)
Other:
- note added: "CORTEX DEBUG CONNECTOR"
- moved on the sheet: C1, C2, C6, C7, JP1, P4, U1, X1
